File: RP2040_HOT-PI/RP2040.kicad_pcb (KiCad board)
At the start: 2 copper layers, 21 x 51 mm, 33 parts, among them J1 USB_C_Receptacle_USB2.0_14P, J2 Conn_01x20, J3 Conn_01x20, J4 Conn_01x03, SW1 SW_Push, U1 RP2040, U3 W25Q128JVS, U4 MCP1700x-330xxTT, Y1 12 MHz

Commit message: Added custom silkscreen
Parts:
- added G***: LOGO, custom-silkscreen:hot-pi-logo, F.Cu at (170.0, 78.2)
- added G***: LOGO, custom-silkscreen:gd-icon, B.Cu at (170.0, 68.8)
Other:
- board text added: "@IvailoKirilov"
